Commit message: update urdf

File: robot_description/urdf/robot.urdf (robot description, URDF)
Before this commit: robot demobot, 3 links, 2 joints
Links:
- added link right_wheel; visual cylinder length=0.025 radius=0.03
- link left_wheel: geometry visual cylinder length=0.025 radius=0.03
Joints:
- added joint right_wheel_joint: type continuous, parent base_link, child right_wheel, origin xyz=0.075 -0.115 -0.01 rpy=1.571 0 0, axis 0 0 1
- joint caster joint: origin xyz=-0.19 0 -0.03 -> xyz=-0.09 0 -0.03
- joint left_wheel_joint: origin xyz=0.05 0.115 -0.01 rpy=1.571 0 0 -> xyz=0.075 0.115 -0.01 rpy=1.571 0 0
