Commit message: create material file

File: robot_description/urdf/robot.urdf.xacro (robot description, xacro)
@@ -1,13 +1,5 @@
 <?xml version="1.0"?>
 <robot xmlns:xacro="http://www.ros.org/wiki/xacro" name="demobot">
-    <material name="black">
-        <color rgba="0 0 0 1"/>
-    </material>
-    <material name="purple">
-        <color rgba="0.3098 0.1765 0.4980 1" />
-    </material>
-    <material name="gray">
-        <color rgba="0.5 0.5 0.5 1" />
-    </material>
+    <xacro:include filename="materials.xacro" />
     <!-- Constants -->
     <xacro:property name="PI" value="3.14159265359" />

Commit message: minor update

File: robot_description/urdf/robot.urdf.xacro (robot description, xacro)
@@ -16,5 +16,5 @@
     <xacro:property name="WHEEL_R" value="0.03" />
     <!-- Wheel macro -->
-    <xacro:macro name="wheel" params="prefix y_reflect">
+    <xacro:macro name="Wheel" params="prefix y_reflect">
         <joint name="${prefix}_wheel_joint" type="continuous">
             <parent link="base_link" />
@@ -53,5 +53,5 @@
         </visual>
     </link>
-    <xacro:wheel prefix="left" y_reflect="1" />
-    <xacro:wheel prefix="right" y_reflect="-1" />
+    <xacro:Wheel prefix="left" y_reflect="1" />
+    <xacro:Wheel prefix="right" y_reflect="-1" />
 </robot>

Commit message: update urdf with physical properties

File: robot_description/urdf/robot.urdf.xacro (robot description, xacro)
@@ -7,7 +7,9 @@
     <xacro:property name="BASE_Y" value="0.2" />
     <xacro:property name="BASE_Z" value="0.005" />
+    <xacro:property name="BASE_M" value="0.2" />
     <xacro:property name="CASTER_OFF_X" value="-0.09" />
     <xacro:property name="CASTER_OFF_Z" value="-0.03" />
     <xacro:property name="CASTER_R" value="0.01" />
+    <xacro:property name="CASTER_M" value="0.1" />
     <xacro:property name="WHEEL_OFF_X" value="0.075" />
     <xacro:property name="WHEEL_OFF_Y" value="0.115" />
@@ -15,5 +17,6 @@
     <xacro:property name="WHEEL_L" value="0.025" />
     <xacro:property name="WHEEL_R" value="0.03" />
-    <!-- Wheel macro -->
+    <xacro:property name="WHEEL_M" value="0.05" />
+    <!-- Macros -->
     <xacro:macro name="Wheel" params="prefix y_reflect">
         <joint name="${prefix}_wheel_joint" type="continuous">
@@ -30,5 +33,29 @@
                 <material name="black" />
             </visual>
+            <collision>
+                <geometry>
+                    <cylinder radius="${WHEEL_R}" length="${WHEEL_L}" />
+                </geometry>
+            </collision>
+            <xacro:CylinderInertial m="${WHEEL_M}" r="${WHEEL_R}" l="${WHEEL_L}" />
         </link>
+    </xacro:macro>
+    <xacro:macro name="BoxInertial" params="m x y z">
+        <inertial>
+            <mass value="${m}" />
+            <inertia ixx="${(m/12) * (z*z + y*y)}" ixy="0.0" ixz="0.0" iyy="${(m/12) * (x*x + z*z)}" iyz="0.0" izz="${(m/12) * (y*y + x*x)}" />
+        </inertial>
+    </xacro:macro>
+    <xacro:macro name="CylinderInertial" params="m r l">
+        <inertial>
+            <mass value="${m}" />
+            <inertia ixx="${(m/12) * (3*r*r + l*l)}" ixy="0" ixz="0" iyy="${(m/12) * (3*r*r + l*l)}" iyz="0" izz="${(m/2) * (r*r)}" />
+        </inertial>
+    </xacro:macro>
+    <xacro:macro name="SphereInertial" params="m r">
+        <inertial>
+            <mass value="${m}" />
+            <inertia ixx="${(2/5) * m * (r*r)}" ixy="0.0" ixz="0.0" iyy="${(2/5) * m * (r*r)}" iyz="0.0" izz="${(2/5) * m * (r*r)}" />
+        </inertial>
     </xacro:macro>
     <!-- Start Modelling -->
@@ -40,4 +67,10 @@
             <material name="purple"/>
         </visual>
+        <collision>
+            <geometry>
+                <box size="${BASE_X} ${BASE_Y} ${BASE_Z}"/>
+            </geometry>
+        </collision>
+        <xacro:BoxInertial m="${BASE_M}" x="${BASE_X}" y="${BASE_Y}" z="${BASE_Z}" />
     </link>
     <joint name="caster joint" type="fixed">
@@ -53,4 +86,10 @@
             <material name="gray"/>
         </visual>
+        <collision>
+            <geometry>
+                <sphere radius="${CASTER_R}"/>
+            </geometry>
+        </collision>
+        <xacro:SphereInertial m="${CASTER_M}" r="${CASTER_R}" />
     </link>
     <xacro:Wheel prefix="left" y_reflect="1" />

Commit message: update gazebo materials

File: robot_description/urdf/robot.urdf.xacro (robot description, xacro)
@@ -40,4 +40,7 @@
             <xacro:CylinderInertial m="${WHEEL_M}" r="${WHEEL_R}" l="${WHEEL_L}" />
         </link>
+        <gazebo reference="${prefix}_wheel_link">
+            <material>Gazebo/Black</material>
+        </gazebo>
     </xacro:macro>
     <xacro:macro name="BoxInertial" params="m x y z">
@@ -74,4 +77,7 @@
         <xacro:BoxInertial m="${BASE_M}" x="${BASE_X}" y="${BASE_Y}" z="${BASE_Z}" />
     </link>
+    <gazebo reference="base_link">
+        <material>Gazebo/Purple</material>
+    </gazebo>
     <joint name="caster joint" type="fixed">
         <parent link="base_link"/>
@@ -93,4 +99,9 @@
         <xacro:SphereInertial m="${CASTER_M}" r="${CASTER_R}" />
     </link>
+    <gazebo reference="caster">
+        <mu1>0.0001</mu1>
+        <mu2>0.0001</mu2>
+        <material>Gazebo/Gray</material>
+    </gazebo>
     <xacro:Wheel prefix="left" y_reflect="1" />
     <xacro:Wheel prefix="right" y_reflect="-1" />

Commit message: add diff drive plugin

File: robot_description/urdf/robot.urdf.xacro (robot description, xacro)
@@ -23,5 +23,5 @@
             <parent link="base_link" />
             <child link="${prefix}_wheel_link" />
-            <origin xyz="${WHEEL_OFF_X} ${y_reflect*WHEEL_OFF_Y} ${WHEEL_OFF_Z}" rpy="${PI/2} 0 0" />
+            <origin xyz="${WHEEL_OFF_X} ${y_reflect*WHEEL_OFF_Y} ${WHEEL_OFF_Z}" rpy="${-PI/2} 0 0" />
             <axis xyz="0 0 1" />
         </joint>
@@ -106,3 +106,27 @@
     <xacro:Wheel prefix="left" y_reflect="1" />
     <xacro:Wheel prefix="right" y_reflect="-1" />
+    <gazebo>
+        <plugin name="differential_drive_controller" filename="libgazebo_ros_diff_drive.so">
+            <!-- <ros>
+                <namespace>/demobot</namespace>
+            </ros> -->
+            <!-- wheels -->
+            <left_joint>left_wheel_joint</left_joint>
+            <right_joint>right_wheel_joint</right_joint>
+            <!-- kinematics -->
+            <wheel_separation>0.23</wheel_separation>
+            <wheel_diameter>0.06</wheel_diameter>
+            <!-- tfs -->
+            <publish_odom>true</publish_odom>
+            <publish_odom_tf>true</publish_odom_tf>
+            <publish_wheel_tf>true</publish_wheel_tf>
+            <odometry_frame>odom</odometry_frame>
+            <!-- limits -->
+            <max_wheel_torque>20</max_wheel_torque>
+            <max_acceleration>1.0</max_acceleration>
+            <!-- miscs -->
+            <robot_base_frame>base_link</robot_base_frame>
+            <update_rate>50</update_rate>
+        </plugin>
+    </gazebo>
 </robot>

Commit message: break down urdf

File: robot_description/urdf/robot.urdf.xacro (robot description, xacro)
@@ -1,190 +1,8 @@
 <?xml version="1.0"?>
 <robot xmlns:xacro="http://www.ros.org/wiki/xacro" name="demobot">
-    <xacro:include filename="materials.xacro" />
-    <!-- Constants -->
-    <xacro:property name="PI" value="3.14159265359" />
-    <xacro:property name="BASE_X" value="0.2" />
-    <xacro:property name="BASE_Y" value="0.2" />
-    <xacro:property name="BASE_Z" value="0.005" />
-    <xacro:property name="BASE_M" value="0.2" />
-    <xacro:property name="CASTER_OFF_X" value="-0.09" />
-    <xacro:property name="CASTER_OFF_Z" value="-0.03" />
-    <xacro:property name="CASTER_R" value="0.01" />
-    <xacro:property name="CASTER_M" value="0.1" />
-    <xacro:property name="WHEEL_OFF_X" value="0.075" />
-    <xacro:property name="WHEEL_OFF_Y" value="0.115" />
-    <xacro:property name="WHEEL_OFF_Z" value="-0.01" />
-    <xacro:property name="WHEEL_L" value="0.025" />
-    <xacro:property name="WHEEL_R" value="0.03" />
-    <xacro:property name="WHEEL_M" value="0.05" />
-    <xacro:property name="LIDAR_R" value="0.035" />
-    <xacro:property name="LIDAR_L" value="0.02" />
-    <xacro:property name="LIDAR_OFF_Z" value="0.08" />
-    <xacro:property name="LIDAR_M" value="0.17" />
-    <!-- Macros -->
-    <xacro:macro name="Wheel" params="prefix y_reflect">
-        <joint name="${prefix}_wheel_joint" type="continuous">
-            <parent link="base_link" />
-            <child link="${prefix}_wheel_link" />
-            <origin xyz="${WHEEL_OFF_X} ${y_reflect*WHEEL_OFF_Y} ${WHEEL_OFF_Z}" rpy="${-PI/2} 0 0" />
-            <axis xyz="0 0 1" />
-        </joint>
-        <link name="${prefix}_wheel_link">
-            <visual>
-                <geometry>
-                    <cylinder radius="${WHEEL_R}" length="${WHEEL_L}" />
-                </geometry>
-                <material name="black" />
-            </visual>
-            <collision>
-                <geometry>
-                    <cylinder radius="${WHEEL_R}" length="${WHEEL_L}" />
-                </geometry>
-            </collision>
-            <xacro:CylinderInertial m="${WHEEL_M}" r="${WHEEL_R}" l="${WHEEL_L}" />
-        </link>
-        <gazebo reference="${prefix}_wheel_link">
-            <material>Gazebo/Black</material>
-        </gazebo>
-    </xacro:macro>
-    <xacro:macro name="BoxInertial" params="m x y z">
-        <inertial>
-            <mass value="${m}" />
-            <inertia ixx="${(m/12) * (z*z + y*y)}" ixy="0.0" ixz="0.0" iyy="${(m/12) * (x*x + z*z)}" iyz="0.0" izz="${(m/12) * (y*y + x*x)}" />
-        </inertial>
-    </xacro:macro>
-    <xacro:macro name="CylinderInertial" params="m r l">
-        <inertial>
-            <mass value="${m}" />
-            <inertia ixx="${(m/12) * (3*r*r + l*l)}" ixy="0" ixz="0" iyy="${(m/12) * (3*r*r + l*l)}" iyz="0" izz="${(m/2) * (r*r)}" />
-        </inertial>
-    </xacro:macro>
-    <xacro:macro name="SphereInertial" params="m r">
-        <inertial>
-            <mass value="${m}" />
-            <inertia ixx="${(2/5) * m * (r*r)}" ixy="0.0" ixz="0.0" iyy="${(2/5) * m * (r*r)}" iyz="0.0" izz="${(2/5) * m * (r*r)}" />
-        </inertial>
-    </xacro:macro>
-    <!-- Start Modelling -->
-    <link name="base_link">
-        <visual>
-            <geometry>
-                <box size="${BASE_X} ${BASE_Y} ${BASE_Z}"/>
-            </geometry>
-            <material name="purple"/>
-        </visual>
-        <collision>
-            <geometry>
-                <box size="${BASE_X} ${BASE_Y} ${BASE_Z}"/>
-            </geometry>
-        </collision>
-        <xacro:BoxInertial m="${BASE_M}" x="${BASE_X}" y="${BASE_Y}" z="${BASE_Z}" />
-    </link>
-    <gazebo reference="base_link">
-        <material>Gazebo/Purple</material>
-    </gazebo>
-    <joint name="caster joint" type="fixed">
-        <parent link="base_link"/>
-        <child link="caster"/>
-        <origin xyz="${CASTER_OFF_X} 0 ${CASTER_OFF_Z}"/>
-    </joint>
-    <link name="caster">
-        <visual>
-            <geometry>
-                <sphere radius="${CASTER_R}"/>
-            </geometry>
-            <material name="gray"/>
-        </visual>
-        <collision>
-            <geometry>
-                <sphere radius="${CASTER_R}"/>
-            </geometry>
-        </collision>
-        <xacro:SphereInertial m="${CASTER_M}" r="${CASTER_R}" />
-    </link>
-    <gazebo reference="caster">
-        <mu1>0.0001</mu1>
-        <mu2>0.0001</mu2>
-        <material>Gazebo/Gray</material>
-    </gazebo>
-    <xacro:Wheel prefix="left" y_reflect="1" />
-    <xacro:Wheel prefix="right" y_reflect="-1" />
-    <gazebo>
-        <plugin name="differential_drive_controller" filename="libgazebo_ros_diff_drive.so">
-            <!-- <ros>
-                <namespace>/demobot</namespace>
-            </ros> -->
-            <!-- wheels -->
-            <left_joint>left_wheel_joint</left_joint>
-            <right_joint>right_wheel_joint</right_joint>
-            <!-- kinematics -->
-            <wheel_separation>0.23</wheel_separation>
-            <wheel_diameter>0.06</wheel_diameter>
-            <!-- tfs -->
-            <publish_odom>true</publish_odom>
-            <publish_odom_tf>true</publish_odom_tf>
-            <publish_wheel_tf>true</publish_wheel_tf>
-            <odometry_frame>odom</odometry_frame>
-            <!-- limits -->
-            <max_wheel_torque>20</max_wheel_torque>
-            <max_acceleration>1.0</max_acceleration>
-            <!-- miscs -->
-            <robot_base_frame>base_link</robot_base_frame>
-            <update_rate>100</update_rate>
-        </plugin>
-    </gazebo>
-    <joint name="lidar_joint" type="fixed">
-        <parent link="base_link" />
-        <child link="lidar" />
-        <origin xyz="0 0 ${(BASE_Z+LIDAR_L)/2+LIDAR_OFF_Z}" />
-    </joint>
-    <link name="lidar">
-        <visual>
-            <geometry>
-                <cylinder radius="${LIDAR_R}" length="${LIDAR_L}" />
-            </geometry>
-            <material name="blue" />
-        </visual>
-        <collision>
-            <geometry>
-                <cylinder radius="${LIDAR_R}" length="${LIDAR_L}" />
-            </geometry>
-        </collision>
-        <xacro:CylinderInertial m="${LIDAR_M}" r="${LIDAR_R}" l="${LIDAR_L}" />
-    </link>
-    <gazebo reference="lidar">
-        <material>Gazebo/Blue</material>
-        <sensor name="lidar" type="ray">
-            <always_on>true</always_on>
-            <visualize>true</visualize>
-            <update_rate>5</update_rate>
-            <ray>
-                <scan>
-                    <horizontal>
-                        <samples>360</samples>
-                        <resolution>1.000000</resolution>
-                        <min_angle>0.000000</min_angle>
-                        <max_angle>6.280000</max_angle>
-                    </horizontal>
-                </scan>
-                <range>
-                    <min>0.120000</min>
-                    <max>6</max>
-                    <resolution>0.015000</resolution>
-                </range>
-                <noise>
-                    <type>gaussian</type>
-                    <mean>0.0</mean>
-                    <stddev>0.01</stddev>
-                </noise>
-            </ray>
-            <plugin name="scan" filename="libgazebo_ros_ray_sensor.so">
-                <ros>
-                    <remapping>~/out:=scan</remapping>
-                </ros>
-                <output_type>sensor_msgs/LaserScan</output_type>
-                <frame_name>lidar</frame_name>
-            </plugin>
-        </sensor>
-    </gazebo>
+    <!-- <xacro:include filename="$(find hpr_description)/urdf/hpr_core.urdf.xacro" /> -->
+    <xacro:include filename="robot_core.xacro" />
+    <!-- <xacro:include filename="lidar.urdf.xacro" />
+    <xacro:include filename="gazebo_ros_diff_drive.xacro" />
+    <xacro:include filename="gazebo_ros_ray.xacro" /> -->
 </robot>

Commit message: separate lidar

File: robot_description/urdf/robot.urdf.xacro (robot description, xacro)
@@ -3,5 +3,4 @@
     <xacro:include filename="robot_core.xacro" />
     <xacro:include filename="gazebo_diff_drive_plugin.xacro" />
-    <!-- <xacro:include filename="lidar.urdf.xacro" />
-    <xacro:include filename="gazebo_ros_ray.xacro" /> -->
+    <xacro:include filename="lidar.xacro" />
 </robot>

File: robot_description/urdf/robot_core.xacro (robot description, xacro)
@@ -21,8 +21,4 @@
     <xacro:property name="WHEEL_R" value="0.03" />
     <xacro:property name="WHEEL_M" value="0.05" />
-    <xacro:property name="LIDAR_R" value="0.035" />
-    <xacro:property name="LIDAR_L" value="0.02" />
-    <xacro:property name="LIDAR_OFF_Z" value="0.08" />
-    <xacro:property name="LIDAR_M" value="0.17" />
     <!-- Macros -->
     <xacro:macro name="Wheel" params="prefix y_reflect">
