Commit message: add lidar and world

File: robot_description/urdf/materials.xacro (robot description, xacro)
@@ -16,4 +16,7 @@
         <color rgba="0 0 0.5 1" />
     </material>
+    <material name="blue">
+        <color rgba="0 0 1 1" />
+    </material>
     <material name="gray">
         <color rgba="0.5 0.5 0.5 1" />

File: robot_description/urdf/robot.urdf.xacro (robot description, xacro)
@@ -18,4 +18,8 @@
     <xacro:property name="WHEEL_R" value="0.03" />
     <xacro:property name="WHEEL_M" value="0.05" />
+    <xacro:property name="LIDAR_R" value="0.035" />
+    <xacro:property name="LIDAR_L" value="0.02" />
+    <xacro:property name="LIDAR_OFF_Z" value="0.08" />
+    <xacro:property name="LIDAR_M" value="0.17" />
     <!-- Macros -->
     <xacro:macro name="Wheel" params="prefix y_reflect">
@@ -130,3 +134,57 @@
         </plugin>
     </gazebo>
+    <joint name="lidar_joint" type="fixed">
+        <parent link="base_link" />
+        <child link="lidar" />
+        <origin xyz="0 0 ${(BASE_Z+LIDAR_L)/2+LIDAR_OFF_Z}" />
+    </joint>
+    <link name="lidar">
+        <visual>
+            <geometry>
+                <cylinder radius="${LIDAR_R}" length="${LIDAR_L}" />
+            </geometry>
+            <material name="blue" />
+        </visual>
+        <collision>
+            <geometry>
+                <cylinder radius="${LIDAR_R}" length="${LIDAR_L}" />
+            </geometry>
+        </collision>
+        <xacro:CylinderInertial m="${LIDAR_M}" r="${LIDAR_R}" l="${LIDAR_L}" />
+    </link>
+    <gazebo reference="lidar">
+        <material>Gazebo/Blue</material>
+        <sensor name="lidar" type="ray">
+            <always_on>true</always_on>
+            <visualize>true</visualize>
+            <update_rate>5</update_rate>
+            <ray>
+                <scan>
+                    <horizontal>
+                        <samples>360</samples>
+                        <resolution>1.000000</resolution>
+                        <min_angle>0.000000</min_angle>
+                        <max_angle>6.280000</max_angle>
+                    </horizontal>
+                </scan>
+                <range>
+                    <min>0.120000</min>
+                    <max>6</max>
+                    <resolution>0.015000</resolution>
+                </range>
+                <noise>
+                    <type>gaussian</type>
+                    <mean>0.0</mean>
+                    <stddev>0.01</stddev>
+                </noise>
+            </ray>
+            <plugin name="scan" filename="libgazebo_ros_ray_sensor.so">
+                <ros>
+                    <remapping>~/out:=scan</remapping>
+                </ros>
+                <output_type>sensor_msgs/LaserScan</output_type>
+                <frame_name>lidar</frame_name>
+            </plugin>
+        </sensor>
+    </gazebo>
 </robot>

Commit message: add camera link and plugin

File: robot_description/urdf/materials.xacro (robot description, xacro)
@@ -19,4 +19,7 @@
         <color rgba="0 0 1 1" />
     </material>
+    <material name="green">
+        <color rgba="0 1 0 1" />
+    </material>
     <material name="gray">
         <color rgba="0.5 0.5 0.5 1" />

File: robot_description/urdf/robot.urdf.xacro (robot description, xacro)
@@ -4,3 +4,4 @@
     <xacro:include filename="gazebo_diff_drive_plugin.xacro" />
     <xacro:include filename="lidar.xacro" />
+    <xacro:include filename="camera.xacro" />
 </robot>
