Commit message: fix viewing angle

File: robot_description/urdf/camera.xacro (robot description, xacro)
@@ -6,5 +6,5 @@
     <xacro:property name="CAM_OFF_X" value="0.1" />
     <xacro:property name="CAM_OFF_Z" value="0.05" />
-    <xacro:property name="CAM_M" value="0.17" />
+    <xacro:property name="CAM_M" value="0.005" />
     <joint name="camera_joint" type="fixed">
         <parent link="base_link" />
@@ -26,5 +26,12 @@
         <xacro:CylinderInertial m="${CAM_M}" r="${CAM_R}" l="${CAM_L}" />
     </link>
-    <gazebo reference="camera">
+    <joint name="lens_joint" type="fixed">
+        <parent link="camera" />
+        <child link="lens" />
+        <origin xyz="0 0 0" rpy="0 ${PI/2} 0"/>
+    </joint>
+    <link name="lens">
+    </link>
+    <gazebo reference="lens">
         <material>Gazebo/Green</material>
         <sensor name="rgb_camera" type="camera">

Commit message: update camera

File: robot_description/urdf/camera.xacro (robot description, xacro)
@@ -26,4 +26,7 @@
         <xacro:CylinderInertial m="${CAM_M}" r="${CAM_R}" l="${CAM_L}" />
     </link>
+    <gazebo reference="camera">
+        <material>Gazebo/Green</material>
+    </gazebo>
     <joint name="lens_joint" type="fixed">
         <parent link="camera" />
@@ -31,12 +34,10 @@
         <origin xyz="0 0 0" rpy="0 ${PI/2} 0"/>
     </joint>
-    <link name="lens">
-    </link>
+    <link name="lens" />
     <gazebo reference="lens">
-        <material>Gazebo/Green</material>
         <sensor name="rgb_camera" type="camera">
             <always_on>true</always_on>
             <visualize>true</visualize>
-            <update_rate>20.0</update_rate>
+            <update_rate>30.0</update_rate>
             <camera name="rgb_camera">
                 <horizontal_fov>1.3962634</horizontal_fov>

Commit message: clean up urdf

File: robot_description/urdf/camera.xacro (robot description, xacro)
@@ -53,7 +53,4 @@
                 <noise>
                   <type>gaussian</type>
-                  <!-- Noise is sampled independently per pixel on each frame.
-                       That pixel's noise value is added to each of its color
-                       channels, which at that point lie in the range [0,1]. -->
                   <mean>0.0</mean>
                   <stddev>0.007</stddev>
@@ -69,20 +66,6 @@
             </camera>
             <plugin name="camera_plugin" filename="libgazebo_ros_camera.so">
-                <!-- Change namespace, camera name and topics so -
-                     * Images are published to: /custom_ns/custom_camera/custom_image
-                     * Camera info is published to: /custom_ns/custom_camera/custom_info
-                -->
-                <!-- <ros>
-                  <namespace>custom_ns</namespace>
-                  <remapping>image_raw:=custom_img</remapping>
-                  <remapping>camera_info:=custom_info</remapping>
-                </ros> -->
-                <!-- Set camera name. If empty, defaults to sensor name (i.e. "sensor_name") -->
-                <!-- <camera_name>custom_camera</camera_name> -->
-                <!-- Set TF frame name. If empty, defaults to link name (i.e. "link_name") -->
-                <!-- <frame_name>custom_frame</frame_name> -->
                 <hack_baseline>0.07</hack_baseline>
-                <!-- No need to repeat distortion parameters or to set autoDistortion -->
-              </plugin>
+                  </plugin>
         </sensor>
     </gazebo>

File: robot_description/urdf/gazebo_diff_drive_plugin.xacro (robot description, xacro)
@@ -3,7 +3,4 @@
     <gazebo>
         <plugin name="differential_drive_controller" filename="libgazebo_ros_diff_drive.so">
-            <!-- <ros>
-                <namespace>/demobot</namespace>
-            </ros> -->
             <!-- wheels -->
             <left_joint>left_wheel_joint</left_joint>

File: robot_description/urdf/robot_core.xacro (robot description, xacro)
@@ -1,6 +1,4 @@
 <?xml version="1.0"?>
 <robot xmlns:xacro="http://www.ros.org/wiki/xacro" >
-    <!-- <xacro:include filename="$(find hpr_description)/urdf/materials.xacro" />
-    <xacro:include filename="$(find hpr_description)/urdf/inertia.xacro" /> -->
     <xacro:include filename="materials.xacro" />
     <xacro:include filename="inertial.xacro" />
@@ -71,5 +69,5 @@
     </joint>
     <link name="base_footprint"/>
-    <joint name="caster joint" type="fixed">
+    <joint name="caster_joint" type="fixed">
         <parent link="base_link"/>
         <child link="caster"/>
