Commit message: increase base_link mass and decrease max wheel torque

File: robot_description/urdf/gazebo_diff_drive_plugin.xacro (robot description, xacro)
@@ -15,5 +15,5 @@
             <odometry_frame>odom</odometry_frame>
             <!-- limits -->
-            <max_wheel_torque>20</max_wheel_torque>
+            <max_wheel_torque>10</max_wheel_torque>
             <max_acceleration>1.0</max_acceleration>
             <!-- miscs -->

File: robot_description/urdf/robot_core.xacro (robot description, xacro)
@@ -8,5 +8,5 @@
     <xacro:property name="BASE_Y" value="0.2" />
     <xacro:property name="BASE_Z" value="0.005" />
-    <xacro:property name="BASE_M" value="0.2" />
+    <xacro:property name="BASE_M" value="2" />
     <xacro:property name="CASTER_OFF_X" value="-0.09" />
     <xacro:property name="CASTER_OFF_Z" value="-0.03" />
