Commit message: update imu location

File: robot_description/urdf/imu.xacro (robot description, xacro)
@@ -4,5 +4,4 @@
     <xacro:property name="IMU_Y" value="0.035" />
     <xacro:property name="IMU_Z" value="0.002" />
-    <xacro:property name="IMU_OFF_X" value="0.075" />
     <xacro:property name="IMU_OFF_Z" value="0.01" />
     <xacro:property name="IMU_M" value="0.005" />
@@ -10,5 +9,5 @@
         <parent link="base_link" />
         <child link="imu" />
-        <origin xyz="${IMU_OFF_X} 0 ${(BASE_Z+IMU_Z)/2+IMU_OFF_Z}" />
+        <origin xyz="0 0 ${(BASE_Z+IMU_Z)/2+IMU_OFF_Z}" />
     </joint>
     <link name="imu">
