Commit message: update robot dimensions

File: demobot_description/urdf/demobot.urdf (robot description, URDF)
Before this commit: robot demobot, 4 links, 3 joints
Links:
- removed link caster
- added link caster_ball; visual sphere radius=0.2
- link base_link: geometry visual box size=1 0.8 0.6
- link left_wheel: geometry visual cylinder length=0.2 radius=0.4
- link right_wheel: geometry visual cylinder length=0.2 radius=0.4
Joints:
- removed joint caster joint
- added joint caster_joint: type fixed, parent base_link, child caster_ball, origin xyz=-0.3 0 -0.3
- joint left_wheel_joint: origin xyz=0.075 0.115 -0.01 rpy=1.571 0 0 -> xyz=0.1 0.5 -0.1 rpy=1.571 0 0
- joint right_wheel_joint: origin xyz=0.075 -0.115 -0.01 rpy=1.571 0 0 -> xyz=0.1 -0.5 -0.1 rpy=1.571 0 0

Commit message: update robot dimensions

File: demobot_description/urdf/demobot.urdf (robot description, URDF)
Before this commit: robot demobot, 4 links, 3 joints
Links:
- link base_link: geometry visual box size=1 0.8 0.4
- link caster_ball: geometry visual sphere radius=0.1
- link left_wheel: geometry visual cylinder length=0.1 radius=0.3
- link right_wheel: geometry visual cylinder length=0.1 radius=0.3
Joints:
- joint caster_joint: origin xyz=-0.3 0 -0.3 -> xyz=-0.4 0 -0.2
- joint left_wheel_joint: origin xyz=0.1 0.5 -0.1 rpy=1.571 0 0 -> xyz=0.2 0.5 0.0 rpy=1.571 0 0
- joint right_wheel_joint: origin xyz=0.1 -0.5 -0.1 rpy=1.571 0 0 -> xyz=0.2 -0.5 0.0 rpy=1.571 0 0
