Commit message: update with new package names

File: demobot_description/urdf/camera.xacro (robot description, xacro)
@@ -4,11 +4,11 @@
     <xacro:property name="CAM_R" value="0.00425" />
     <xacro:property name="CAM_L" value="0.001" />
-    <xacro:property name="CAM_OFF_X" value="0.1" />
-    <xacro:property name="CAM_OFF_Z" value="0.05" />
+    <xacro:property name="CAM_OFF_X" value="0.5" />
+    <xacro:property name="CAM_OFF_Z" value="0.3" />
     <xacro:property name="CAM_M" value="0.005" />
     <joint name="camera_joint" type="fixed">
         <parent link="base_link" />
         <child link="camera" />
-        <origin xyz="${CAM_OFF_X} 0 ${BASE_Z/2+CAM_R+CAM_OFF_Z}" rpy="0 ${-PI/2} 0"/>
+        <origin xyz="${CAM_OFF_X} 0 ${CAM_OFF_Z}" rpy="0 ${-PI/2} 0"/>
     </joint>
     <link name="camera">
@@ -69,20 +69,6 @@
             </camera>
             <plugin name="camera_plugin" filename="libgazebo_ros_camera.so">
-                <!-- Change namespace, camera name and topics so -
-                     * Images are published to: /custom_ns/custom_camera/custom_image
-                     * Camera info is published to: /custom_ns/custom_camera/custom_info
-                -->
-                <!-- <ros>
-                  <namespace>custom_ns</namespace>
-                  <remapping>image_raw:=custom_img</remapping>
-                  <remapping>camera_info:=custom_info</remapping>
-                </ros> -->
-                <!-- Set camera name. If empty, defaults to sensor name (i.e. "sensor_name") -->
-                <!-- <camera_name>custom_camera</camera_name> -->
-                <!-- Set TF frame name. If empty, defaults to link name (i.e. "link_name") -->
-                <!-- <frame_name>custom_frame</frame_name> -->
                 <hack_baseline>0.07</hack_baseline>
-                <!-- No need to repeat distortion parameters or to set autoDistortion -->
-              </plugin>
+            </plugin>
         </sensor>
     </gazebo>

File: demobot_description/urdf/demobot.urdf.xacro (robot description, xacro)
@@ -6,3 +6,4 @@
     <xacro:include filename="gazebo_diff_drive_plugin.xacro" />
     <xacro:include filename="lidar.xacro" />
+    <xacro:include filename="camera.xacro" />
 </robot>
