Commit message: breakdown urdf

File: demobot_description/urdf/demobot.urdf.xacro (robot description, xacro)
@@ -1,191 +1,8 @@
 <?xml version="1.0"?>
 <robot xmlns:xacro="http://www.ros.org/wiki/xacro" name="demobot">
-    <xacro:include filename="materials.xacro" />
-    <!-- Constants -->
-    <xacro:property name="PI" value="3.14159265359" />
-    <xacro:property name="BASE_X" value="1.0" />
-    <xacro:property name="BASE_Y" value="0.8" />
-    <xacro:property name="BASE_Z" value="0.4" />
-    <xacro:property name="BASE_M" value="4" />
-    <xacro:property name="CASTER_OFF_X" value="-0.4" />
-    <xacro:property name="CASTER_OFF_Z" value="-0.2" />
-    <xacro:property name="CASTER_R" value="0.1" />
-    <xacro:property name="CASTER_M" value="1.0" />
-    <xacro:property name="WHEEL_OFF_X" value="0.2" />
-    <xacro:property name="WHEEL_OFF_Y" value="0.5" />
-    <xacro:property name="WHEEL_R" value="0.3" />
-    <xacro:property name="WHEEL_L" value="0.1" />
-    <xacro:property name="WHEEL_M" value="0.5" />
-    <xacro:property name="LIDAR_OFF_Z" value="0.35" />
-    <xacro:property name="LIDAR_R" value="0.035" />
-    <xacro:property name="LIDAR_L" value="0.02" />
-    <xacro:property name="LIDAR_M" value="0.17" />
-    <!-- Inertial matrix macro -->
-    <xacro:macro name="BoxInertial" params="m x y z">
-        <inertial>
-            <mass value="${m}" />
-            <inertia ixx="${(m/12) * (z*z + y*y)}" ixy="0.0" ixz="0.0" iyy="${(m/12) * (x*x + z*z)}" iyz="0.0" izz="${(m/12) * (y*y + x*x)}" />
-        </inertial>
-    </xacro:macro>
-    <xacro:macro name="CylinderInertial" params="m r l">
-        <inertial>
-            <mass value="${m}" />
-            <inertia ixx="${(m/12) * (3*r*r + l*l)}" ixy="0" ixz="0" iyy="${(m/12) * (3*r*r + l*l)}" iyz="0" izz="${(m/2) * (r*r)}" />
-        </inertial>
-    </xacro:macro>
-    <xacro:macro name="SphereInertial" params="m r">
-        <inertial>
-            <mass value="${m}" />
-            <inertia ixx="${(2/5) * m * (r*r)}" ixy="0.0" ixz="0.0" iyy="${(2/5) * m * (r*r)}" iyz="0.0" izz="${(2/5) * m * (r*r)}" />
-        </inertial>
-    </xacro:macro>
-    <!-- Wheel macro -->
-    <xacro:macro name="Wheel" params="prefix y_reflect">
-        <joint name="${prefix}_wheel_joint" type="continuous">
-            <parent link="base_link" />
-            <child link="${prefix}_wheel" />
-            <origin xyz="${WHEEL_OFF_X} ${y_reflect*WHEEL_OFF_Y} 0" rpy="${-PI/2} 0 0" />
-            <axis xyz="0 0 1" />
-        </joint>
-        <link name="${prefix}_wheel">
-            <visual>
-                <geometry>
-                    <cylinder radius="${WHEEL_R}" length="${WHEEL_L}" />
-                </geometry>
-                <material name="black" />
-            </visual>
-            <collision>
-                <geometry>
-                    <cylinder radius="${WHEEL_R}" length="${WHEEL_L}" />
-                </geometry>
-            </collision>
-            <xacro:CylinderInertial m="${WHEEL_M}" r="${WHEEL_R}" l="${WHEEL_L}" />
-        </link>
-        <gazebo reference="${prefix}_wheel">
-            <material>Gazebo/Black</material>
-        </gazebo>
-    </xacro:macro>
-    <!-- Start Modelling -->
-    <link name="base_link">
-        <visual>
-            <geometry>
-                <box size="${BASE_X} ${BASE_Y} ${BASE_Z}"/>
-            </geometry>
-            <material name="purple"/>
-        </visual>
-        <collision>
-            <geometry>
-                <box size="${BASE_X} ${BASE_Y} ${BASE_Z}"/>
-            </geometry>
-        </collision>
-        <xacro:BoxInertial m="${BASE_M}" x="${BASE_X}" y="${BASE_Y}" z="${BASE_Z}" />
-    </link>
-    <gazebo reference="base_link">
-        <material>Gazebo/Purple</material>
-    </gazebo>
-    <joint name="caster_joint" type="fixed">
-        <parent link="base_link"/>
-        <child link="caster_ball"/>
-        <origin xyz="${CASTER_OFF_X} 0 ${CASTER_OFF_Z}"/>
-    </joint>
-    <link name="caster_ball">
-        <visual>
-            <geometry>
-                <sphere radius="${CASTER_R}"/>
-            </geometry>
-            <material name="gray"/>
-        </visual>
-        <collision>
-            <geometry>
-                <sphere radius="${CASTER_R}"/>
-            </geometry>
-        </collision>
-        <xacro:SphereInertial m="${CASTER_M}" r="${CASTER_R}" />
-    </link>
-    <gazebo reference="caster_ball">
-        <material>Gazebo/Gray</material>
-        <mu1>0.0001</mu1>
-        <mu2>0.0001</mu2>
-    </gazebo>
-    <xacro:Wheel prefix="left" y_reflect="1" />
-    <xacro:Wheel prefix="right" y_reflect="-1" />
-    <!-- Diff drive plugin -->
-    <gazebo>
-        <plugin name="differential_drive_controller" filename="libgazebo_ros_diff_drive.so">
-            <!-- <ros>
-                <namespace>/demobot</namespace>
-            </ros> -->
-            <!-- wheels -->
-            <left_joint>left_wheel_joint</left_joint>
-            <right_joint>right_wheel_joint</right_joint>
-            <!-- kinematics -->
-            <wheel_separation>1.0</wheel_separation>
-            <wheel_diameter>0.6</wheel_diameter>
-            <!-- tfs -->
-            <publish_odom>true</publish_odom>
-            <publish_odom_tf>true</publish_odom_tf>
-            <publish_wheel_tf>true</publish_wheel_tf>
-            <odometry_frame>odom</odometry_frame>
-            <!-- limits -->
-            <max_wheel_torque>20</max_wheel_torque>
-            <max_acceleration>1.0</max_acceleration>
-            <!-- miscs -->
-            <robot_base_frame>base_link</robot_base_frame>
-            <update_rate>100</update_rate>
-        </plugin>
-    </gazebo>
-    <joint name="lidar_joint" type="fixed">
-        <parent link="base_link" />
-        <child link="lidar" />
-        <origin xyz="0 0 ${LIDAR_OFF_Z}" />
-    </joint>
-    <link name="lidar">
-        <visual>
-            <geometry>
-                <cylinder radius="${LIDAR_R}" length="${LIDAR_L}" />
-            </geometry>
-            <material name="blue" />
-        </visual>
-        <collision>
-            <geometry>
-                <cylinder radius="${LIDAR_R}" length="${LIDAR_L}" />
-            </geometry>
-        </collision>
-        <xacro:CylinderInertial m="${LIDAR_M}" r="${LIDAR_R}" l="${LIDAR_L}" />
-    </link>
-    <gazebo reference="lidar">
-        <material>Gazebo/Blue</material>
-        <sensor name="lidar" type="ray">
-            <always_on>true</always_on>
-            <visualize>true</visualize>
-            <update_rate>5</update_rate>
-            <ray>
-                <scan>
-                    <horizontal>
-                        <samples>360</samples>
-                        <resolution>1.000000</resolution>
-                        <min_angle>0.000000</min_angle>
-                        <max_angle>6.280000</max_angle>
-                    </horizontal>
-                </scan>
-                <range>
-                    <min>0.120000</min>
-                    <max>6</max>
-                    <resolution>0.015000</resolution>
-                </range>
-                <noise>
-                    <type>gaussian</type>
-                    <mean>0.0</mean>
-                    <stddev>0.01</stddev>
-                </noise>
-            </ray>
-            <plugin name="scan" filename="libgazebo_ros_ray_sensor.so">
-                <ros>
-                    <remapping>~/out:=scan</remapping>
-                </ros>
-                <output_type>sensor_msgs/LaserScan</output_type>
-                <frame_name>lidar</frame_name>
-            </plugin>
-        </sensor>
-    </gazebo>
+    <xacro:include filename="material.xacro" />
+    <xacro:include filename="inertial.xacro" />
+    <xacro:include filename="core.xacro" />
+    <xacro:include filename="gazebo_diff_drive_plugin.xacro" />
+    <xacro:include filename="lidar.xacro" />
 </robot>

File: demobot_description/urdf/material.xacro (robot description, xacro)
@@ -16,4 +16,10 @@
         <color rgba="0 0 0.5 1" />
     </material>
+    <material name="blue">
+        <color rgba="0 0 1 1" />
+    </material>
+    <material name="green">
+        <color rgba="0 1 0 1" />
+    </material>
     <material name="gray">
         <color rgba="0.5 0.5 0.5 1" />

Commit message: update packages

File: demobot_description/urdf/demobot.urdf.xacro (robot description, xacro)
@@ -7,3 +7,4 @@
     <xacro:include filename="lidar.xacro" />
     <xacro:include filename="camera.xacro" />
+    <xacro:include filename="imu.xacro" />
 </robot>

File: demobot_description/urdf/imu.xacro (robot description, xacro)
@@ -4,5 +4,4 @@
     <xacro:property name="IMU_Y" value="0.035" />
     <xacro:property name="IMU_Z" value="0.002" />
-    <xacro:property name="IMU_OFF_X" value="0.075" />
     <xacro:property name="IMU_OFF_Z" value="0.01" />
     <xacro:property name="IMU_M" value="0.005" />
@@ -10,5 +9,5 @@
         <parent link="base_link" />
         <child link="imu" />
-        <origin xyz="${IMU_OFF_X} 0 ${(BASE_Z+IMU_Z)/2+IMU_OFF_Z}" />
+        <origin xyz="0 0 ${(BASE_Z+IMU_Z)/2+IMU_OFF_Z}" />
     </joint>
     <link name="imu">
